File: PCB/Nice-Buoy-V1.0/untitled.kicad_sch (KiCad schematic)
At the start: 34 parts, among them J206 MainswitchLeds, J207 BalanceConnector, Q201 AO3401A, Q202 AO3401A, Q203 AO3401A, Q204 AO3401A, Q205 AO3401A, Q206 AO3401A, Q207 AO3401A, Q208 AO3401A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

Commit message: Many changes in schematics
Parts:
- removed Q207, Q208: AO3401A, symbol Simulation_SPICE:PMOS
- removed R104 (x2): 100k, symbol Device:R_Small
- removed R108 (x2): 100, symbol Device:R_Small
- added C25: 100n, A_Device:C_0603, symbol Device:C_Small
- added D6: GREEN, symbol Device:LED_Small
- added D7: RED, symbol Device:LED_Small
- added J10: SW1, Connector_JST:JST_XH_B2B-XH-A_1x02_P2.50mm_Vertical, symbol Connector:Conn_01x02_Socket
- added J11: SW2, Connector_JST:JST_XH_B2B-XH-A_1x02_P2.50mm_Vertical, symbol Connector:Conn_01x02_Socket
- added J12: SW3, Connector_JST:JST_XH_B2B-XH-A_1x02_P2.50mm_Vertical, symbol Connector:Conn_01x02_Socket
- added J13: LED1, Connector_JST:JST_XH_B2B-XH-A_1x02_P2.50mm_Vertical, symbol Connector:Conn_01x02_Socket
- added J14: LED2, Connector_JST:JST_XH_B2B-XH-A_1x02_P2.50mm_Vertical, symbol Connector:Conn_01x02_Socket
- added J15: LED3, Connector_JST:JST_XH_B2B-XH-A_1x02_P2.50mm_Vertical, symbol Connector:Conn_01x02_Socket
- added R104 (x2): 4.7k, A_Device:R_0603, symbol Device:R_Small
- added R106 (x3): 100, A_Device:R_0603, symbol Device:R_Small
- added R106 (x2): 1k, A_Device:R_0603, symbol Device:R_Small
- added U8: ADS1110A0, Package_TO_SOT_SMD:SOT-23-6, symbol Analog_ADC:ADS1110
- C22: renamed from C216; footprint (none) -> A_Device:C_0603
- J16: renamed from J206; footprint (none) -> Connector_JST:JST_XH_B3B-XH-A_1x03_P2.50mm_Vertical; LCSC (none) -> C161870
- J9: renamed from J207; footprint (none) -> Connector_JST:JST_XH_B7B-XH-A_1x07_P2.50mm_Vertical; LCSC (none) -> C144398
- Q1: renamed from Q201; footprint (none) -> A_IC_SOT:SC-59_1.6x3_P0.95
- Q2: renamed from Q202; footprint (none) -> A_IC_SOT:SC-59_1.6x3_P0.95
- Q3: renamed from Q203; footprint (none) -> A_IC_SOT:SC-59_1.6x3_P0.95
- Q4: renamed from Q204; footprint (none) -> A_IC_SOT:SC-59_1.6x3_P0.95
- Q5: renamed from Q205; footprint (none) -> A_IC_SOT:SC-59_1.6x3_P0.95
- Q6: renamed from Q206; footprint (none) -> A_IC_SOT:SC-59_1.6x3_P0.95
- R104, R105, R106, R108: footprint (none) -> A_Device:R_0603
- TP1: renamed from TP201; footprint (none) -> A_Pads_Pins:Testpoint_0.6x1.0
- renumbered U204 to U6, U206 to U7
Connections:
- net +3.3V: now also U8.5 (VDD)
- net +3V3: now also C25.1
- net GND: now also C25.2, J10.1 (Pin_1), J11.1 (Pin_1), J12.1 (Pin_1), J13.1 (Pin_1), J14.1 (Pin_1), J15.1 (Pin_1), U8.2 (GND), U8.6 (VIN-)
- net GREEN: now also J16.1 (Pin_1), R104.1; no longer J16.3 (Pin_3)
- net RED: now also J16.3 (Pin_3), R104.1; no longer J16.1 (Pin_1)
- net at U7.11 (O8): now also R104.2
- net at U7.12 (O7): now also R104.2
- net at C22.1, D107.2 (A), R105.2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: now also U8.1 (VIN+)
- net SCL: now reaches U6.12 (SCK)
- net SCL: now also U8.3 (SCL)
- net SDA: now reaches U6.13 (SDA)
- net SDA: now also U8.4 (SDA)
- net SW1: now reaches U6.21 (GPA0)
- net SW1: now also J10.2 (Pin_2)
- net SW2: now reaches U6.22 (GPA1)
- net SW2: now also J11.2 (Pin_2)
- net SW3: now reaches U6.23 (GPA2)
- net SW3: now also J12.2 (Pin_2)
- net LED1: now reaches U6.24 (GPA3)
- net LED1: now also R106.1
- net LED2: now reaches U6.25 (GPA4)
- net LED2: now also R106.1
- net LED3: now reaches U6.26 (GPA5)
- net LED3: now also R106.1
- net at U6.27 (GPA6): now also R106.1
- net at U6.28 (GPA7): now also R106.1
- net +12V renamed +28V
- net +28V: now also Q1.3 (S), R104.1, U7.10 (COM)
- removed net S6: J9.7 (Pin_7), Q1.3 (S), R104.1, U7.10 (COM)
- new net: D7.1 (K), R106.2
- new net: J13.2 (Pin_2), R106.2
- new net: J15.2 (Pin_2), R106.2
- new net: D6.1 (K), R106.2
- new net: J14.2 (Pin_2), R106.2
- new net +5V: D6.2 (A), D7.2 (A)
- no-connect marks 2 -> 3
Other:
- note added: "0x48"
- note removed: "To adc"
- moved on the sheet: C22, D107, J16, TP1
