File: PCB/Nice-Buoy-V1.0/Accumonitor.kicad_sch (KiCad schematic)
At the start: 45 parts, among them J10 SW1, J11 SW2, J12 SW3, J13 LED1, J14 LED2, J15 LED3, J16 MainswitchLeds, J9 BalanceConnector, Q4 AO3401A, Q5 AO3401A, Q6 AO3401A, Q7 AO3401A, Q8 AO3401A, Q9 AO3401A, U7 MCP23017_SS, U8 ULN2803A, U9 ADS1110A0

Commit message: Battery monitor not working
Parts:
- added D703, D704, D705, D706, D707: 1N4148WS, A_Device:D_SOD-323_1.8x1.4x1.15, symbol Device:D_Small
- renumbered C34 to C703, D12 to D701, D13 to D702, J9 to J701, J10 to J702, J11 to J703, J12 to J704, J13 to J705, J14 to J706, J15 to J707, J16 to J708, Q4 to Q701, Q5 to Q702, Q6 to Q703, Q7 to Q704, Q8 to Q705, Q9 to Q706, TP2 to TP701, U7 to U701, U8 to U702, U9 to U703
Other:
- moved on the sheet: Q701, Q702, Q703, Q704, Q705, Q706, R104

Commit message: Routing finnished
Parts:
- removed D703, D704, D705, D706, D707: 1N4148WS, A_Device:D_SOD-323_1.8x1.4x1.15, symbol Device:D_Small
- removed J701: BalanceConnector, Connector_JST:JST_XH_B7B-XH-A_1x07_P2.50mm_Vertical, symbol Connector:Conn_01x07_Pin
- removed Q701, Q702, Q703, Q704, Q705, Q706: AO3401A, A_IC_SOT:SC-59_1.6x3_P0.95, symbol Simulation_SPICE:PMOS
- removed R104 (x6): 100k, A_Device:R_0603, symbol Device:R_Small
- removed R106 (x5): 1.5k, A_Device:R_0603, symbol Device:R_Small
- removed U702: ULN2803A, A_IC_SOP:SO-18_7.5x11.6_P50mil, symbol Transistor_Array:ULN2803A
- removed U703: ADS1110A0, Package_TO_SOT_SMD:SOT-23-6, symbol Analog_ADC:ADS1110
- added J707: 3.3V switch, Connector_PinHeader_2.54mm:PinHeader_1x02_P2.54mm_Vertical, symbol Connector:Conn_01x02_Socket
- added J708: Vbatt switch, Connector_PinHeader_2.54mm:PinHeader_1x02_P2.54mm_Vertical, symbol Connector:Conn_01x02_Socket
- added Q701, Q702, Q703, Q704: MMBT5551L, Package_TO_SOT_SMD:SOT-23, symbol Transistor_BJT:MMBT5551L
- added R106 (x2): 100, A_Device:R_0603, symbol Device:R_Small
- added R108 (x4): 1k, A_Device:R_0603, symbol Device:R_Small
- added TP702: T1, A_Pads_Pins:Testpoint_0.4x0.7, symbol Connector:TestPoint
- added TP703: T2, A_Pads_Pins:Testpoint_0.4x0.7, symbol Connector:TestPoint
- J705: renamed from J703; value SW2 -> SW3
- J706: renamed from J704; value SW3 -> SW2
- R105: value 1k -> 6.2k
- renumbered J705 to J701, J706 to J702, J707 to J703, J702 to J704, J708 to J709
Connections:
- net +5V is gone; now on net +3.3V: D701.2 (A), D702.2 (A)
- net +28V: now also R105.1, R106.1
- net +3.3V: now also R106.1
- net GND: now also Q701.2 (E), Q702.2 (E), Q703.2 (E), Q704.2 (E)
- net RED: now also R104.2; no longer R104.1
- net SW1: now also U701.23 (GPA2); no longer U701.21 (GPA0)
- net SW2: now also J706.2 (Pin_2); no longer J705.2 (Pin_2)
- net SW3: now also J705.2 (Pin_2), U701.21 (GPA0); no longer J706.2 (Pin_2), U701.23 (GPA2)
- net at U701.1 (GPB0): now also R108.1
- net at R104.2: now also Q702.3 (C)
- net at U701.2 (GPB1): now also R108.1
- net at U701.3 (GPB2): now also R108.1
- net at U701.4 (GPB3): now also R108.1
- net at U701.5 (GPB4): now also TP702.1
- net at U701.6 (GPB5): now also TP703.1
- net Vbatt: now reaches C703.1, D107.2 (A), R105.2, R108.1, R108.1, TP701.1
- new net: Q701.1 (B), R108.2
- new net: J707.1 (Pin_1), Q701.3 (C)
- new net: Q702.1 (B), R108.2
- new net: Q703.3 (C), R104.1
- new net: Q703.1 (B), R108.2
- new net: Q704.1 (B), R108.2
- new net: J707.2 (Pin_2), R106.2
- new net: J708.2 (Pin_2), R106.2
- new net: J708.1 (Pin_1), Q704.3 (C)
- no-connect marks 3 -> 4
Other:
- note added: "LIPO info nominal cel voltage 3.7 max cel voltage 4.2 S6 nominal voltage 22.2V Max 25.2 Cut off 19.2V"
- note removed: "0x48"
- note removed: "12.6"
- note removed: "16.8"
- note removed: "21"
- note removed: "25.2"
- note removed: "4.2"
- note removed: "8.4"
- note removed: "LIPO info nominal cel voltage 3.7 max cel voltage 4.2 S6 nominal voltage 22.2V Max 25.2 Cut off 19.2V 4.2 8.4 12.6 16.8 21 25.2"
- note removed: "uref 2.8 I 0.01 S1 4.2 S2 8.4 S3 12.6 S4 16.8 S5 21.0 S6 25.2 Sn = 1.5*uref*n"
- moved on the sheet: C703, D107, J701, J702, J703, J704, J705, J706, J709, R104, R105, R106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
