File: PCB/Nice-Buoy-V1_0/Nice-Buoy-V1_0.kicad_pcb (KiCad board)
At the start: 4 copper layers, 100 x 80 mm, 154 parts, among them J101 USB_B_Mini, J102 LEDSTRIP, J103 Display, J201 Accu, J202 ESC SB POWER, J203 ESC BB POWER, J401 ESC-BB, J402 ESC-SB, J501 GPS, J601 Conn_Coaxial, J701 LED1, J702 LED2, J703 LED3, J704 SW1, J705 SW3, J706 SW2, J707 3.3V switch, J708 Vbatt switch, J709 MainswitchLeds, J901 Display, Q101 2N7002, Q102 2N7002, Q201 NCE01P30K, Q701 MMBT5551L, Q702 MMBT5551L, Q703 MMBT5551L, Q704 MMBT5551L, SW101 ~{BOOT}, SW102 ~{RESET}, SW103 SW_SPST, SW104 SW2, SW201 ON/OFF, U101 SRV05-4, U102 CP2104-F03-GMR, U103 ESP32-WROOM-32E_(visible_peri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, U201 AP7363, U202 XL1509-5.0E1, U301 LSM303C, U601 Ai-Thinker-Ra-01, U701 MCP23017_SS, U801 LIS2HH12

Commit message: PCB finished and orderd at JLCPCB
Parts:
- removed SW103: SW_SPST, Connector_PinHeader_2.54mm:PinHeader_1x02_P2.54mm_Vertical
- removed SW104: SW2, Connector_PinHeader_2.54mm:PinHeader_1x02_P2.54mm_Vertical
- removed TP101: RW1, A_Misc:ReworkPins
- removed TP102: RW2, A_Misc:ReworkPins
- added C113: 1n, A_Device:C_0603, F.Cu at (125.3, 82.4)
- added C114: 1n, A_Device:C_0603, F.Cu at (125.0, 91.3)
- added J104: SW1, Connector_JST:JST_XH_B3B-XH-A_1x03_P2.50mm_Vertical, F.Cu at (134.7, 76.8)
- added J105: SW2, Connector_JST:JST_XH_B3B-XH-A_1x03_P2.50mm_Vertical, F.Cu at (134.7, 88.0)
- added R113: 100, A_Device:R_0603, F.Cu at (127.6, 81.6)
- added R114: 100, A_Device:R_0603, F.Cu at (127.6, 90.5)
- added R119: 100, A_Device:R_0603, F.Cu at (127.6, 85.9)
- added R120: 100, A_Device:R_0603, F.Cu at (127.6, 92.0)
- added TP1: RW1, A_Misc:ReworkPins, F.Cu at (125.3, 55.9)
- added TP2: RW2, A_Misc:ReworkPins, F.Cu at (125.3, 66.0)
- D201: value SM4007PL -> ZMM5V6-M; footprint A_Device:D_SOD-123_2.85x1.8x1.3 -> A_Device:D_MiniMELF
- J101: value USB_B_Mini -> 1051330011; footprint Connector_USB:USB_Micro-B_Amphenol_10118193-0001LF_Horizontal -> Connector_USB:USB_Micro-B_Molex-105133-0001
- moved U103 10.2 mm to (105.5, 115.0), turned to 180 degrees
- moved C801 5.79 mm to (129.9, 76.3), turned to 90 degrees
- moved R117 4.57 mm to (127.6, 84.4)
- moved R118 4.57 mm to (127.6, 82.9)
- moved J102 3.12 mm to (138.1, 68.4)
- moved R115 3.08 mm to (127.6, 87.4)
- moved R116 3.08 mm to (127.6, 88.9)
- moved C802 2.90 mm to (126.6, 76.0)
- moved C110 2.37 mm to (124.5, 79.3)
- moved C803 2.37 mm to (126.6, 79.3)
- moved U801 2.37 mm to (129.1, 79.3)
- moved J101 1.92 mm to (129.2, 112.0)
- moved C601 1.52 mm to (121.2, 80.1)
- moved C602 1.52 mm to (121.2, 83.6)
- renumbered C113 to C115, J103 to J102, J102 to J103, R113 to R115, R114 to R116, R115 to R117, R116 to R118, R117 to R121
Connections:
- R115 pad 1: Net-(SW104-A) -> Net-(J105-Pin_2)
- R116 pad 2: Net-(SW104-A) -> Net-(J105-Pin_2)
- R117 pad 1: Net-(SW103-A) -> Net-(J104-Pin_2)
- R118 pad 2: Net-(SW103-A) -> Net-(J104-Pin_2)
- U103 pad 4: Net-(SW103-A) -> Net-(U103-GPIO36)
- U103 pad 5: Net-(SW104-A) -> Net-(U103-GPIO39)
Routing:
- net Net-(SW103-A): track 34.6 -> 0.00 mm, vias 2 -> 0
- net Net-(U103-GPIO36): track 0.00 -> 34.6 mm, vias 0 -> 2
- net Net-(SW104-A): track 30.4 -> 0.00 mm, vias 2 -> 0
- net Net-(U103-GPIO39): track 0.00 -> 25.7 mm, vias 0 -> 2
- net Net-(J104-Pin_1): track 0.00 -> 21.7 mm
- net Net-(J104-Pin_3): track 0.00 -> 19.6 mm
- net Net-(J104-Pin_2): track 0.00 -> 10.1 mm
- net Net-(J105-Pin_2): track 0.00 -> 9.47 mm
- net +3.3V: track 135.3 -> 129.8 mm
- net +5V: track 164.5 -> 170.0 mm, vias 3 -> 1
- net GND: track 334.3 -> 338.8 mm, vias 167 -> 166
- net /CPU/SCL: track 142.6 -> 139.9 mm
- net Net-(J101-D+): track 16.4 -> 18.9 mm
- net DR0: track 49.2 -> 51.3 mm
- net /CPU/SDA: track 149.9 -> 147.9 mm, vias 4 -> 3
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Other:
- board text added: "LORA"
