File: PCB/Nice-Buoy-V1_0/OledDispaly.kicad_sch (KiCad schematic)
At the start: 2 parts, among them J901 Display

Commit message: PCB finished and orderd at JLCPCB
Parts:
- J901: now not fitted; now left out of the parts list
Changed lines of the file:
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@@
     (pin "1")
     (instances
-      (project "Nice-Buoy-V1.0"
+      (project "Nice-Buoy-V1_0"
         (path "/77bea089-a6ae-4a6f-b95b-7a9010ad7c5d/b5739766-77e3-499c-9625-6fbf43d3f159"
           (reference "#PWR0902") (unit 1)
@@
     (pin "1")
     (instances
-      (project "Nice-Buoy-V1.0"
+      (project "Nice-Buoy-V1_0"
         (path "/77bea089-a6ae-4a6f-b95b-7a9010ad7c5d/b4716c37-6296-4cc3-83d4-c08b9373ace7"
           (reference "#PWR0121") (unit 1)
@@
   )
   (symbol (lib_id "Connector:Conn_01x04_Socket") (at 146.05 78.74 0) (unit 1)
-    (in_bom yes) (on_board yes) (dnp no) (fields_autoplaced)
+    (in_bom no) (on_board yes) (dnp yes) (fields_autoplaced)
     (property "Reference" "J901" (at 147.32 78.74 0)
       (effects (font (size 1.27 1.27)) (justify left))
@@
     (pin "4")
     (instances
-      (project "Nice-Buoy-V1.0"
+      (project "Nice-Buoy-V1_0"
         (path "/77bea089-a6ae-4a6f-b95b-7a9010ad7c5d/b5739766-77e3-499c-9625-6fbf43d3f159"
           (reference "J901") (unit 1)
@@
     (pin "1")
     (instances
-      (project "Nice-Buoy-V1.0"
+      (project "Nice-Buoy-V1_0"
         (path "/77bea089-a6ae-4a6f-b95b-7a9010ad7c5d/b5739766-77e3-499c-9625-6fbf43d3f159"
           (reference "#PWR0901") (unit 1)
@@
     (pin "1")
     (instances
-      (project "Nice-Buoy-V1.0"
+      (project "Nice-Buoy-V1_0"
         (path "/77bea089-a6ae-4a6f-b95b-7a9010ad7c5d/20fb3964-c9d0-4636-b697-42bcddc45d6f"
           (reference "#PWR02") (unit 1)
@@
         )
       )
-      (project "Nice-Buoy-V1.0"
+      (project "Nice-Buoy-V1_0"
         (path "/77bea089-a6ae-4a6f-b95b-7a9010ad7c5d/015165a8-30a1-4680-bca0-c8d83aec4be2"
           (reference "C20") (unit 1)
