File: PCB/Nice-Buoy-V1_0/PSU_sch.kicad_sch (KiCad schematic)
At the start: 32 parts, among them J201 Accu, J202 ESC SB POWER, J203 ESC BB POWER, Q201 NCE01P30K, SW201 ON/OFF, U201 AP7363, U202 XL1509-5.0E1

Commit message: Working version!
Other:
- note added: "Not suited for the job"
Changed lines of the file:
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@@
+		)
+	)
+	(text "Not suited for the job"
+		(exclude_from_sim no)
+		(at 161.544 109.474 0)
+		(effects
+			(font
+				(size 1.27 1.27)
+			)
 		)
 	)
