File: PCB/Robuoy-Sub-V1_0/PSU_sch.kicad_sch (KiCad schematic)
At the start: 69 parts, among them J201 Accu, J202 LoadbalanceAccu1, J203 LoadbalanceAccu2, J204 CHARGE/ON-OFF, J205 PWR_Charger, J206 LoadbalanceCharger, J207 ESCSB, J208 ESCBB, Q201 AO3400A, Q202 AO3400A, Q203 AO3400A, Q204 AO3400A, Q205 AO3400A, Q206 AO3400A, Q207 AO3400A, Q208 AO3400A, SW201 SS-12D11-G050/On-Off, U201 TPS5430DDAR, U202 SN74LV1T34DBV, U203 SN74LV1T34DBV, U204 TLV61046ADB

Commit message: PCB changed
Parts:
- removed SW201: SS-12D11-G050/On-Off, A_Connector:SS-12D10L5, symbol Switch:SW_DPST_x2
- added SW201: On/Off, A_Connector:SS-12D10L5, symbol NicE:SW_slide_SP
Connections:
- net +VSW: now also SW201.2
- net Vbatt: now also SW201.1
Changed lines of the file:
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@@
 	(wire
 		(pts
+			(xy 39.37 116.84) (xy 57.15 116.84)
+		)
+		(stroke
+			(width 0)
+			(type default)
+		)
+	)
+	(wire
+		(pts
 			(xy 45.72 88.9) (xy 60.96 88.9)
 		)
@@
 	(wire
 		(pts
+			(xy 34.29 114.3) (xy 34.29 116.84)
+		)
+		(stroke
+			(width 0)
+			(type default)
+		)
+	)
+	(wire
+		(pts
 			(xy 121.92 190.5) (xy 130.81 190.5)
 		)
@@
 	(wire
 		(pts
-			(xy 44.45 116.84) (xy 57.15 116.84)
+			(xy 39.37 114.3) (xy 39.37 116.84)
 		)
 		(stroke
@@
 	)
 	(symbol
+		(lib_id "NicE:SW_slide_SP")
+		(at 39.37 111.76 90)
+		(unit 1)
+		(exclude_from_sim no)
+		(in_bom yes)
+		(on_board yes)
+		(dnp no)
+		(property "Reference" "SW201"
+			(at 36.322 119.38 90)
+			(effects
+				(font
+					(size 1.27 1.27)
+				)
+			)
+		)
+		(property "Value" "On/Off"
+			(at 36.83 108.712 90)
+			(effects
+				(font
+					(size 1.27 1.27)
+				)
+			)
+		)
+		(property "Footprint" "A_Connector:SS-12D10L5"
+			(at 39.37 109.22 0)
+			(effects
+				(font
+					(size 1.27 1.27)
+				)
+				(hide yes)
+			)
+		)
+		(property "Datasheet" ""
+			(at 39.37 109.22 0)
+			(effects
+				(font
+					(size 1.27 1.27)
+				)
+				(hide yes)
+			)
+		)
+		(property "Description" ""
+			(at 39.37 109.22 0)
+			(effects
+				(font
+					(size 1.27 1.27)
+				)
+				(hide yes)
+			)
+		)
+		(property "LCSC" "C319012"
+			(at 39.37 111.76 0)
+			(effects
+				(font
+					(size 1.27 1.27)
+				)
+				(hide yes)
+			)
+		)
+		(pin "1"
+		)
+		(pin "3"
+		)
+		(pin "2"
+		)
+		(instances
+			(project "Robuoy-Sub"
+				(path "/77bea089-a6ae-4a6f-b95b-7a9010ad7c5d/b4716c37-6296-4cc3-83d4-c08b9373ace7"
+					(reference "SW201")
+					(unit 1)
+				)
+			)
+		)
+	)
+	(symbol
 		(lib_name "+3.3V_1")
 		(lib_id "power:+3.3V")
@@
 					(unit 1)
 				)
-			)
-		)
-	)
-	(symbol
-		(lib_id "Switch:SW_DPST_x2")
-		(at 39.37 116.84 0)
-		(unit 1)
-		(exclude_from_sim no)
-		(in_bom yes)
-		(on_board yes)
-		(dnp no)
-		(fields_autoplaced yes)
-		(property "Reference" "SW201"
-			(at 39.37 110.49 0)
-			(effects
-				(font
-					(size 1.27 1.27)
-				)
-			)
-		)
-		(property "Value" "SS-12D11-G050/On-Off"
-			(at 39.37 113.03 0)
-			(effects
-				(font
-					(size 1.27 1.27)
-				)
-			)
-		)
-		(property "Footprint" "A_Connector:SS-12D10L5"
-			(at 39.37 116.84 0)
-			(effects
-				(font
-					(size 1.27 1.27)
-				)
-				(hide yes)
-			)
-		)
-		(property "Datasheet" "https://wmsc.lcsc.com/wmsc/upload/file/pdf/v2/lcsc/2110151630_XKB-Connection-SS-12D10L5_C319012.pdf"
-			(at 39.37 116.84 0)
-			(effects
-				(font
-					(size 1.27 1.27)
-				)
-				(hide yes)
-			)
-		)
-		(property "Description" "Single Pole Single Throw (SPST) switch, separate symbol"
-			(at 39.37 116.84 0)
-			(effects
-				(font
-					(size 1.27 1.27)
-				)
-				(hide yes)
-			)
-		)
-		(property "LCSC" "C319012"
-			(at 39.37 116.84 90)
-			(effects
-				(font
-					(size 1.27 1.27)
-				)
-				(hide yes)
-			)
-		)
-		(pin "4"
-		)
-		(pin "2"
-		)
-		(pin "1"
-		)
-		(pin "3"
-		)
-		(instances
-			(project "Robuoy-Sub"
-				(path "/77bea089-a6ae-4a6f-b95b-7a9010ad7c5d/b4716c37-6296-4cc3-83d4-c08b9373ace7"
-					(reference "SW201")
-					(unit 1)
-				)

Commit message: Pcb edditing
Parts:
- removed J206: LoadbalanceCharger, Connector_JST:JST_XH_B7B-XH-A_1x07_P2.50mm_Vertical, symbol Connector:Conn_01x07_Socket
- added R209, R211: 100, A_Device:R_0603, symbol Device:R_Small
- J201: value Accu -> Accu 1
- J205: value PWR_Charger -> Accu 2; footprint A_Connector:AMASS_XT60-F_1x02_P7.20mm_Vertical -> A_Connector:AMASS_XT60-M_1x02_P7.20mm_Vertical
- renumbered R209 to R210, R210 to R212, R211 to R213, TP206 to TP202, TP208 to TP203, TP207 to TP204, TP202 to TP205, TP203 to TP206, TP210 to TP207, TP209 to TP208, TP204 to TP209, TP205 to TP210
Connections:
- net +VSW: now also J204.5 (Pin_5); no longer J204.8 (Pin_8)
- net GND: now also J204.3 (Pin_3), J204.4 (Pin_4); no longer J204.10 (Pin_10), J204.9 (Pin_9)
- net Vbatt: now also J204.1 (Pin_1), J204.2 (Pin_2); no longer J204.11 (Pin_11), J204.12 (Pin_12)
- net at Q202.1 (G), Q204.1 (G), Q206.1 (G)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: now also R211.1; no longer U203.4 (Y)
- net at Q201.1 (G), Q203.1 (G), Q205.1 (G)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: now also R209.1; no longer U202.4 (Y)
- net at J202.1 (Pin_1), J203.1 (Pin_1): now also J204.12 (Pin_12); no longer J204.1 (Pin_1)
- net at J202.2 (Pin_2), J203.2 (Pin_2): now also J204.11 (Pin_11); no longer J204.2 (Pin_2)
- net at J202.3 (Pin_3), J203.3 (Pin_3): now also J204.10 (Pin_10); no longer J204.3 (Pin_3)
- net at J202.4 (Pin_4), J203.4 (Pin_4): now also J204.9 (Pin_9); no longer J204.4 (Pin_4)
- net at J202.5 (Pin_5), J203.5 (Pin_5): now also J204.8 (Pin_8); no longer J204.5 (Pin_5)
- net at J202.6 (Pin_6), J203.6 (Pin_6): now also J204.7 (Pin_7); no longer J204.6 (Pin_6)
- net at J202.7 (Pin_7), J203.7 (Pin_7): now also J204.6 (Pin_6); no longer J204.7 (Pin_7)
- new net: R211.2, U203.4 (Y)
- new net: R209.2, U202.4 (Y)
Other:
- moved on the sheet: U202, U203
