File: PCB/Robobuoy-Top-V2_0/Robobuoy-Top-V2_0.kicad_pcb (KiCad board)
At the start: 4 copper layers, 65 x 69 mm, 112 parts, among them J101 PROG/JTAG, J102 Option_Buttons, J103 FRONT SWITCH, J104 GPS, J105 I2C Option, J201 Charge/On_Off, J202 Accu, Q101 A03401A, Q102 AO3400A, Q202 A03401A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

Commit message: Pc programm starting to code
Parts:
- removed D205: 5V, A_Device:LED_0805
- removed L202: 10uH, A_Device:FTC252012S
- removed R212: 51K, A_Device:R_0603
- removed R213: 16K, A_Device:R_0603
- removed R215: 1.5K, A_Device:R_0603
- removed TP201, TP206: 0.795V, A_Pads_Pins:Testpad_1.4
- removed TP202: 5V, A_Pads_Pins:Testpoint_0.9x1.5
- removed TP207: 3V3, A_Pads_Pins:Testpad_1.4
- removed U204: TLV61046ADB, Package_TO_SOT_SMD:SOT-23-6
- added C211: 10u/10V, A_Passive:C_0805, F.Cu at (48.6, 27.5)
- added C212: 10u/10V, A_Passive:C_0805, F.Cu at (48.6, 30.4)
- added C213: 10u/10V, A_Passive:C_0805, F.Cu at (48.6, 33.3)
- added C214: 100n, A_Device:C_0603, F.Cu at (52.9, 32.5)
- added C215: 100n, A_Device:C_0603, F.Cu at (52.9, 34.9)
- added C216: 10u/10V, A_Passive:C_0805, F.Cu at (48.6, 36.2)
- added C217: 10u/10V, A_Passive:C_0805, F.Cu at (48.6, 39.1)
- added U203: TPS63020DSJR, A_Confocal:QFN14_1, F.Cu at (76.5, 58.4)
- C204, C208: value 4.7uF -> 10u/10V; footprint A_Device:C_1206_(1.6) -> A_Passive:C_0805
- C205: value 100n -> 10u/10V; footprint A_Device:C_0603 -> A_Passive:C_0805
- L201: value 10uH -> 1.5uH / 3.7A; footprint A_Device:FTC252012S -> A_Passive:L_2x2.5
- R216: value 1K -> 4.7K
- U201: value TLV61046ADB -> LM1117MP-3.3/TR; footprint Package_TO_SOT_SMD:SOT-23-6 -> Package_TO_SOT_SMD:SOT-223
- moved L201 41.5 mm to (76.5, 54.7), turned to 0 degrees
- moved U201 39.7 mm to (74.0, 65.8)
Connections:
- C201 pad 1: VBUS -> Net-(U203-PS/SYNC)
- C204 pad 1: +5V -> VBUS
- C208 pad 1: +3.3V -> +5V
- L201 pad 1: VBUS -> Net-(L201-Pad1)
- L201 pad 2: Net-(U201-SW) -> Net-(L201-Pad2)
- Q202 pad 1: VBUS -> Net-(J202-Pin_2)
- Q202 pad 3: Net-(J202-Pin_2) -> VBUS
- U201 pad 1: Net-(U201-SW) -> GND
- U201 pad 2: GND -> Net-(U201-VO)
- U201 pad 3: Net-(U201-FB) -> +5V
- U201 pad 4: Enable -> (no net)
Routing:
- net +3.3V: track 260.4 -> 211.4 mm, vias 10 -> 8
- net VBUS: track 114.7 -> 97.0 mm
- net +5V: track 132.8 -> 121.5 mm
- net GND: track 128.8 -> 117.8 mm
- net Net-(U204-FB): track 9.23 -> 0.00 mm, vias 2 -> 0
- net Net-(U201-FB): track 9.48 -> 1.65 mm, vias 2 -> 0
- net Enable: track 107.0 -> 102.2 mm
- net Net-(J202-Pin_2): track 29.2 -> 31.5 mm
- net Net-(U204-SW): track 2.23 -> 0.00 mm
- net Net-(U201-SW): track 2.23 -> 0.00 mm
- net Net-(D205-A): track 1.32 -> 0.00 mm
- net PAD: track 54.6 -> 55.5 mm
