File: PCB/Robobuoy-Sub-v2_0/CPU_sch.kicad_sch (KiCad schematic)
At the start: 66 parts, among them J101 PROG/JTAG, J102 PUSH BUTTON, J103 RS232_Option, J104 ESC_BB, J105 ESC_SB, J106 Compass, Q101 AO3400A, Q102 AO3400A, SW103 MODE, SW3 ~{BOOT}, SW4 ~{RESET}, U101 ESP32-WROOM-32E_(visible_peri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, U102 USBLC6-4SC6, U103 LSM303AGRTR, U104 LTC4311, U105 SN74LV1T34DBV, U106 SN74LV1T34DBV

Commit message: Many changes again :)
Parts:
- removed C115: 100n, A_Device:C_0603, symbol Device:C_Small
- removed J103: RS232_Option, Connector_PinSocket_2.54mm:PinSocket_1x04_P2.54mm_Vertical, symbol Connector:Conn_01x04_Pin
- removed J106: Compass, Connector_JST:JST_XH_B4B-XH-A_1x04_P2.50mm_Vertical, symbol Connector:Conn_01x04_Socket
- removed JP101: 5V/3.3V, Jumper:SolderJumper-3_P1.3mm_Bridged12_RoundedPad1.0x1.5mm, symbol Jumper:SolderJumper_3_Bridged12
- removed TP102: RXD, A_Pads_Pins:Testpad_1, symbol Connector:TestPoint_Small
- removed TP103: TXD, A_Pads_Pins:Testpad_1, symbol Connector:TestPoint_Small
- removed U104: LTC4311, Package_TO_SOT_SMD:Texas_R-PDSO-G6, symbol NicE:LTC4311
- added R103, R114: 100, A_Device:R_0603, symbol Device:R_Small
- D106: value PWR_ESC_BB -> PWR_ESC_SB
- R109, R110: value 1.8k -> 4.7k
- U102: now fitted
Connections:
- net +5V: no longer C110.1, C111.1, U105.5 (VCC), U106.5 (VCC)
- net ESC_BB: now also R103.2; no longer TP107.1, U105.2 (A)
- net ESC_SB: now also R114.2; no longer TP108.1, U106.2 (A)
- net GND: no longer C110.2, C111.2
- net at J104.2 (Pin_2), R109.2: now also C111.1, U105.5 (VCC)
- net at J104.3 (Pin_3), R111.2: now also C111.2
- net at J105.3 (Pin_3), R112.2: now also C110.2
- net at J105.2 (Pin_2), R110.2: now also C110.1, U106.5 (VCC)
- net SCL: no longer names the net of R105.2, TP104.1, U101.36 (SCL/GPIO22), U102.6 (I/O4), U103.1 (SCL/SPC)
- net SDA: no longer names the net of R104.2, TP105.1, U101.33 (SDA/GPIO21), U102.4 (I/O3), U103.4 (SDA/SDI/SDO)
- new net: R114.1, TP108.1, U106.2 (A)
- new net: R103.1, TP107.1, U105.2 (A)
Other:
- moved on the sheet: BZ101, C110, C111, D102, D105, D106, Q102, R108, R109, R110, R111, R112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

Commit message: Struct re defined. not finished yet
Parts:
- removed D102: 1N4148WS, A_Device:D_SOD-323_1.8x1.4x1.15, symbol Device:D_Small
- removed J102: PUSH BUTTON, Connector_JST:JST_XH_B3B-XH-A_1x03_P2.50mm_Vertical, symbol Connector:Conn_01x03_Pin
- removed Q101: AO3400A, Package_TO_SOT_SMD:SOT-23, symbol Transistor_FET:2N7002
- removed R106, R107: 100, A_Device:R_0603, symbol Device:R_Small
- added D108: SS14, A_Device:D_SMA_4.3x3x2.4, symbol Device:D_Small
- added TP102, TP103: ESC_5V, A_Pads_Pins:Testpad_1, symbol Connector:TestPoint_Small
- D101: value 1N4148WS -> SS14; footprint A_Device:D_SOD-323_1.8x1.4x1.15 -> A_Device:D_SMA_4.3x3x2.4; LCSC C2128 -> C2480
Connections:
- net +5V is gone; now on net +3.3V: BZ101.1 (+)
- net +3.3V: now also D108.1 (K)
- net BUTTON: now also D108.2 (A); no longer D101.2 (A)
- net GND: no longer D105.1 (K), D106.1 (K), U105.3 (GND), U106.3 (GND)
- net at C111.1, J104.2 (Pin_2), R109.2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: now also TP102.1
- net at C111.2, J104.3 (Pin_3), R111.2: now also D105.1 (K), U105.3 (GND)
- net at BZ101.2 (-), Q102.3 (D): now also D101.2 (A)
- net at C110.2, J105.3 (Pin_3), R112.2: now also D106.1 (K), U106.3 (GND)
- net at C110.1, J105.2 (Pin_2), R110.2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: now also TP103.1
- net COM: now reaches U102.1 (I/O1)
- net COM: now also U101.28 (TXD/GPIO17), U102.3 (I/O2); no longer U101.27 (RXD/GPIO16)
- net BUTTON_LIGHT: no longer names the net of U101.29 (CS/GPIO5)
- new net VbatEn: U101.27 (RXD/GPIO16)
- no-connect marks 10 -> 11
Other:
- moved on the sheet: BZ101, C110, C111, C112, D103, D104, D105, D106, D107, J101, J104, J105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

Commit message: Many changes
Parts:
- removed C110, C111, C114: 100n, A_Device:C_0603, symbol Device:C_Small
- removed D105: PWR_ESC_BB, LED_SMD:LED_0603_1608Metric, symbol Device:LED_Small
- removed D106: PWR_ESC_SB, LED_SMD:LED_0603_1608Metric, symbol Device:LED_Small
- removed D108: SS14, A_Device:D_SMA_4.3x3x2.4, symbol Device:D_Small
- removed J104: ESC_BB, Connector_JST:JST_XH_B3B-XH-A_1x03_P2.50mm_Vertical, symbol Connector:Conn_01x03_Pin
- removed J105: ESC_SB, Connector_JST:JST_XH_B3B-XH-A_1x03_P2.50mm_Vertical, symbol Connector:Conn_01x03_Pin
- removed R103, R111, R112, R114: 100, A_Device:R_0603, symbol Device:R_Small
- removed R109, R110: 4.7k, A_Device:R_0603, symbol Device:R_Small
- removed TP102, TP103: ESC_5V, A_Pads_Pins:Testpad_1, symbol Connector:TestPoint_Small
- removed TP107: ESC_BB, A_Pads_Pins:Testpad_1, symbol Connector:TestPoint_Small
- removed TP108: ESC_SB, A_Pads_Pins:Testpad_1, symbol Connector:TestPoint_Small
- removed U105, U106: SN74LV1T34DBV, Package_TO_SOT_SMD:SOT-23-5, symbol Logic_LevelTranslator:SN74LV1T34DBV
- added C117: 10n, A_Device:C_0603, symbol Device:C_Small
- added J102, J103: Conn_01x03_Pin, Connector_Wire:SolderWire-0.75sqmm_1x03_P4.8mm_D1.25mm_OD2.3mm, symbol Connector:Conn_01x03_Pin
- renumbered C119 to C102, C118 to C103, C117 to C104, C113 to C114, D103 to D101, D104 to D102, D107 to D103, D101 to D105, Q102 to Q101, R113 to R103, R108 to R106, TP106 to TP101, TP101 to TP102, TP105 to TP103, U103 to U102, U102 to U103
Connections:
- net ESC_BB: now also U101.10 (GPIO25), U103.4 (I/O3), J103.2 (Pin_2); no longer U101.26 (D1/GPIO4)
- net ESC_SB: now also U103.6 (I/O4), J102.2 (Pin_2)
- net GND: now also C117.1, J102.1 (Pin_1), J103.1 (Pin_1)
- net at C114.1, C25.1, FB101.2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: now also C117.2
- net at R105.2, TP104.1, U101.36 (SCL/GPIO22)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: no longer U103.6 (I/O4)
- net at R104.2, TP103.1, U101.33 (SDA/GPIO21)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: no longer U103.4 (I/O3)
- net PWR_ESC_BB: no longer names the net of U101.8 (GPIO32)
- net PWR_ESC_SB: no longer names the net of U101.37 (MOSI/GPIO23)
- new net PwrEn: U101.26 (D1/GPIO4)
- new net Vbatt: J102.3 (Pin_3), J103.3 (Pin_3)
- no-connect marks 11 -> 10
Other:
- moved on the sheet: BZ101, C112, D105, Q101, R103, R106, SW103, TP102, U103

Commit message: Pcb changes
Parts:
- removed D102: WS2812B, LED_SMD:LED_WS2812B_PLCC4_5.0x5.0mm_P3.2mm, symbol LED:WS2812B
- removed D105: SS14, A_Device:D_SMA_4.3x3x2.4, symbol Device:D_Small
- removed J102, J103: Conn_01x03_Pin, Connector_Wire:SolderWire-0.75sqmm_1x03_P4.8mm_D1.25mm_OD2.3mm, symbol Connector:Conn_01x03_Pin
- removed R60: 10K, A_Device:R_0603, symbol Device:R
- removed SW3: ~{BOOT}, Connector_PinHeader_2.54mm:PinHeader_1x02_P2.54mm_Vertical, symbol Switch:SW_Push
- added D102: SM4007PL, A_Device:D_SOD-123_2.85x1.8x1.3, symbol Device:D_Small
- added D104: WS2812B, LED_SMD:LED_WS2812B_PLCC4_5.0x5.0mm_P3.2mm, symbol LED:WS2812B
- renumbered C52 to C101, C24 to C105, C24 to C106, C25 to C107, C25 to C108, C25 to C109, C25 to C110, C25 to C111, C25 to C113, C117 to C115, R61 to R102, R106 to R103, R103 to R106, SW4 to SW102
Connections:
- net +3.3V: now also C112.2, R106.1, D102.1 (K), D104.1 (VDD); no longer SW103.2
- net DR0: now also C112.1, R106.2, SW103.2
- net GND: now also SW103.1, D104.3 (VSS); no longer C112.1, R106.2
- net PwrEn: now also U101.27 (RXD/GPIO16); no longer U101.26 (D1/GPIO4)
- net VbatEn: now also U101.26 (D1/GPIO4); no longer U101.27 (RXD/GPIO16)
- net at BZ101.2 (-), Q101.3 (D): now also D102.2 (A)
- net at D101.2 (DOUT): now also D103.4 (DIN)
- net ESC_PWR_BB: now reaches U101.8 (GPIO32)
- net ESC_PWR_SB: now reaches U101.9 (GPIO33)
- net at D103.2 (DOUT): now also D104.4 (DIN)
- removed net BUTTON: C112.2, R106.1, SW103.1, U101.31 (MISO/GPIO19)
Other:
- note added: "Manual reset"
- note removed: "Manual reset / program enable"
- moved on the sheet: C101, C112, R102, R106, SW102, SW103
