File: PCB/Robobuoy-Sub-v2_0/esc.kicad_sch (KiCad schematic)
At the start: 28 parts, among them J401 PWR_ESC_SB, J402 ESC_SB, J404 INPUT_SB, Q401 AO3400A, Q402 AO3401A, Q403 AO3401A, Q404 AO3401A, Q405 AO3401A, Q406 AO3401A, U401 SN74LV1T34DBV

Commit message: Pcb changes
Changed lines of the file:
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@@
 (kicad_sch
-	(version 20231120)
+	(version 20241209)
 	(generator "eeschema")
-	(generator_version "8.0")
+	(generator_version "9.0")
 	(paper "A3")
 	(junction
