File: PCB/Robobuoy-Top-Round-v2_0/Compass_sch.kicad_sch (KiCad schematic)
At the start: 4 parts, among them U301 Ai-Thinker-Ra-02

Commit message: PCP's finsehd for production.
Parts:
- removed C301, C302: 100u/10V, Capacitor_SMD:C_1210_3225Metric, symbol Device:C_Small
- removed C303: 100n, A_Device:C_0603, symbol Device:C_Small
- removed U301: Ai-Thinker-Ra-02, A_Module:Ai-Thinker-Ra-02-LoRa, symbol RF_Module:Ai-Thinker-Ra-02
- added C24: 10u, Capacitor_SMD:C_1210_3225Metric, symbol Device:C_Small
- added C25 (x3): 100n, A_Device:C_0603, symbol Device:C_Small
- added U301: LSM303AGRTR, Package_LGA:LGA-12_2x2mm_P0.5mm, symbol Sensor_Motion:LSM303C
Connections:
- net +3.3V: now also C24.1, C25.1, C25.1, U301.10 (VDDIO), U301.2 (CS_XL), U301.3 (CS_MAG), U301.9 (VDD)
- net GND: now also C24.2, C25.2, C25.2, C25.2, U301.6 (GND), U301.8 (GND)
- new net: C25.1, U301.5 (C1)
- new net SCL: U301.1 (SCL/SPC)
- new net SDA: U301.4 (SDA/SDI/SDO)
- no-connect marks 6 -> 3
Other:
- note added: "Compass"
- note removed: "RADIO_1 MOSI RADIO_2 MISO RADIO_3 SCK RADIO_4 ^CS RADIO_5 ^RESET"
