File: PCB/Robobuoy-Top-Round-v2_0/Robobuoy-Top-Round-v2_0.kicad_sch (KiCad schematic)
At the start: 4 parts

Commit message: PCP's finsehd for production.
Other:
- sheet CPU ports: added COM, ON, RADIO_[1..6], VbatEn, Vsamp; removed RADIO_[1..5], Vbatt
- sheet Lora ports: added RADIO_[1..6]; removed RADIO_[1..5]
- sheet PSU ports: added COM, ON, VbatEn, Vsamp; removed Vbatt
Changed lines of the file:
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@@
+	(wire
+		(pts
+			(xy 119.38 120.65) (xy 119.38 161.29)
+		)
+		(stroke
+			(width 0)
+			(type default)
+		)
+	)
+	(wire
+		(pts
+			(xy 114.3 120.65) (xy 114.3 161.29)
+		)
+		(stroke
+			(width 0)
+			(type default)
+		)
+	)
+	(bus
+		(pts
+			(xy 116.84 41.91) (xy 116.84 50.8)
+		)
+		(stroke
+			(width 0)
+			(type default)
+		)
+	)
 	(wire
 		(pts
@@
 		)
 	)
-	(bus
+	(wire
 		(pts
-			(xy 116.84 41.91) (xy 116.84 50.8)
+			(xy 111.76 120.65) (xy 111.76 161.29)
 		)
 		(stroke
@@
 		)
 		(instances
-			(project "Robuoy-Top"
+			(project "Robobuoy-Top-V2_0"
 				(path "/77bea089-a6ae-4a6f-b95b-7a9010ad7c5d"
 					(reference "H404")
@@
 		)
 		(instances
-			(project "Robuoy-Top"
+			(project "Robobuoy-Top-V2_0"
 				(path "/77bea089-a6ae-4a6f-b95b-7a9010ad7c5d"
 					(reference "H403")
@@
 		)
 		(instances
-			(project "Robuoy-Top"
+			(project "Robobuoy-Top-V2_0"
 				(path "/77bea089-a6ae-4a6f-b95b-7a9010ad7c5d"
 					(reference "H402")
@@
 		)
 		(instances
-			(project "Robuoy-Top"
+			(project "Robobuoy-Top-V2_0"
 				(path "/77bea089-a6ae-4a6f-b95b-7a9010ad7c5d"
 					(reference "H401")
@@
 			)
 		)
-		(pin "RADIO_[1..5]" bidirectional
+		(pin "RADIO_[1..6]" bidirectional
 			(at 116.84 41.91 270)
 			(effects
@@
 		)
 		(instances
-			(project "Robuoy-Top"
+			(project "Robobuoy-Top-Round-v2_0"
 				(path "/77bea089-a6ae-4a6f-b95b-7a9010ad7c5d"
 					(page "6")
@@
 			)
 		)
-		(pin "RADIO_[1..5]" bidirectional
+		(pin "RADIO_[1..6]" bidirectional
 			(at 116.84 50.8 90)
 			(effects
@@
 			)
 		)
-		(pin "Vbatt" output
+		(pin "VbatEn" input
+			(at 114.3 120.65 270)
+			(effects
+				(font
+					(size 1.27 1.27)
+				)
+				(justify left)
+			)
+		)
+		(pin "Vsamp" output
 			(at 116.84 120.65 270)
 			(effects
@@
 			)
 		)
-		(instances
-			(project "Robuoy-Top"
+		(pin "COM" bidirectional
+			(at 119.38 120.65 270)
+			(effects
+				(font
+					(size 1.27 1.27)
+				)
+				(justify left)
+			)
+		)
+		(pin "ON" input
+			(at 111.76 120.65 270)
+			(effects
+				(font
+					(size 1.27 1.27)
+				)
+				(justify left)
+			)
+		)
+		(instances
+			(project "Robobuoy-Top-Round-v2_0"
 				(path "/77bea089-a6ae-4a6f-b95b-7a9010ad7c5d"
 					(page "1")
@@
 			)
 		)
-		(pin "Vbatt" input
+		(pin "VbatEn" output
+			(at 114.3 161.29 90)
+			(effects
+				(font
+					(size 1.27 1.27)
+				)
+				(justify right)
+			)
+		)
+		(pin "Vsamp" input
 			(at 116.84 161.29 90)
 			(effects
@@
 			)
 		)
-		(instances
-			(project "Robuoy-Top"
+		(pin "COM" bidirectional
+			(at 119.38 161.29 90)
+			(effects
+				(font
+					(size 1.27 1.27)
+				)
+				(justify right)
+			)
+		)
+		(pin "ON" output
+			(at 111.76 161.29 90)
+			(effects
+				(font
+					(size 1.27 1.27)
+				)
+				(justify right)
+			)
+		)
+		(instances
+			(project "Robobuoy-Top-Round-v2_0"
 				(path "/77bea089-a6ae-4a6f-b95b-7a9010ad7c5d"
 					(page "2")
