File: PCB/Robobuoy-Top-Round-v2_0/Robobuoy-Top-Round-v2_0.kicad_pcb (KiCad board)
At the start: 4 copper layers, 66 x 52 mm, 81 parts, among them J101 Prog, J103 Conn_01x06_Socket, J104 GPS, J201 CHRG/DATA, J202 CHRG/ON-OFF, Q101 A03401A, Q102 AO3400A, Q201 AO3400A, Q202 AO3401A, SW101 ~{BOOT}/MODE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

Commit message: Serial comms working now
Connections:
- U101 pad 10: LEDS -> BUTTON_LIGHT
- U101 pad 11: BUTTON_LIGHT -> LEDS
- U101 pad 13: /CPU/RADIO_6 -> unconnected-(U101-MTMS/SCK/CLK/GPIO14-Pad13)
- U101 pad 16: unconnected-(U101-MTCK/MOSI/D3/GPIO13-Pad16) -> /CPU/RADIO_5
- U101 pad 23: /CPU/RADIO_5 -> /CPU/RADIO_6
- U101 pad 5: unconnected-(U101-GPIO39-Pad5) -> BUTTON
