File: PCB/Robobuoy-Sub-v2_1_CPU/Robobuoy-Sub-CPU-v2_1.kicad_pcb (KiCad board)
At the start: 4 copper layers, 50 x 42 mm, 59 parts, among them J101 Prog, J103 ESC_BB, J108 TO PSU, Q101 AO3400A, Q102 MMBT3904, Q117 MMBT3904, SW101 ~{RESET}, SW102 MODE, U101 ESP32-WROOM-32E_(visible_peri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, U102 LSM303AGRTR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

Commit message: Some mods
Parts:
- U102: footprint Package_LGA:LGA-12_2x2mm_P0.5mm -> A_Device:LGA-12_2x2mm_P0.5mm
- U104: value LM1117DT-3.3 -> LM1117S-3.3; footprint Package_TO_SOT_SMD:TO-252-3_TabPin2 -> A_IC_SOT:SOT223
Routing:
- net +5V: track 118.3 -> 124.3 mm
- net +3.3V: track 254.9 -> 256.6 mm
