File: PCB/Robobuoy-Sub-v2_1_CPU/Robobuoy-Sub-CPU-v2_1.kicad_sch (KiCad schematic)
At the start: 59 parts, among them J101 Prog, J103 ESC_BB, J108 TO PSU, Q101 AO3400A, Q102 MMBT3904, Q117 MMBT3904, SW101 ~{RESET}, SW102 MODE, U101 ESP32-WROOM-32E_(visible_peri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, U102 LSM303AGRTR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

Commit message: Some mods
Parts:
- J101: LCSC C65114 -> C11214
- U102: footprint Package_LGA:LGA-12_2x2mm_P0.5mm -> A_Device:LGA-12_2x2mm_P0.5mm
- U104: value LM1117DT-3.3 -> LM1117S-3.3; footprint Package_TO_SOT_SMD:TO-252-3_TabPin2 -> A_IC_SOT:SOT223; LCSC (none) -> C126027
Changed lines of the file:
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@@
 			)
 		)
-		(property "LCSC" "C65114"
+		(property "LCSC" "C11214"
 			(at 49.53 26.67 0)
 			(effects
@@
 			)
 		)
-		(property "Footprint" "Package_LGA:LGA-12_2x2mm_P0.5mm"
+		(property "Footprint" "A_Device:LGA-12_2x2mm_P0.5mm"
 			(at 332.74 62.23 0)
 			(effects
@@
 			)
 		)
-		(property "Value" "LM1117DT-3.3"
+		(property "Value" "LM1117S-3.3"
 			(at 130.81 227.33 0)
 			(effects
@@
 			)
 		)
-		(property "Footprint" "Package_TO_SOT_SMD:TO-252-3_TabPin2"
+		(property "Footprint" "A_IC_SOT:SOT223"
 			(at 130.81 231.14 0)
 			(effects
@@
 			)
 		)
-		(property "Datasheet" "http://www.ti.com/lit/ds/symlink/lm1117.pdf"
+		(property "Datasheet" "chrome-extension://efaidnbmnnnibpcajpcglclefindmkaj/https://jlcpcb.com/api/file/downloadByFileSystemAccessId/8586183105745203200"
 			(at 130.81 231.14 0)
 			(effects
@@
 			)
 		)
-		(property "Description" "800mA Low-Dropout Linear Regulator, 3.3V fixed output, TO-252"
+		(property "Description" "1A Low-Dropout Linear Regulator, 3.3V fixed output, TO-223"
+			(at 130.81 231.14 0)
+			(effects
+				(font
+					(size 1.27 1.27)
+				)
+				(hide yes)
+			)
+		)
+		(property "LCSC" "C126027"
 			(at 130.81 231.14 0)
 			(effects

Commit message: Loads of cahnges. Serial working stabile now (one resistor hardware mod) Ack hadled correct now. Less lora messsages
Other:
- note added: "Make 1K"
Changed lines of the file:
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@@
+		)
+	)
+	(text "Make 1K"
+		(exclude_from_sim no)
+		(at 78.232 154.432 0)
+		(effects
+			(font
+				(size 1.27 1.27)
+			)
 		)
 	)
