File: PCB/Robobuoy-Top-v2_1/Lora.kicad_sch (KiCad schematic)
At the start: 4 parts, among them U301 Ai-Thinker-Ra-02

Commit message: New pcb's done
Other:
- moved on the sheet: C303
Changed lines of the file:
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@@
 	)
 	(junction
-		(at 128.905 182.88)
+		(at 129.54 177.8)
+		(diameter 0)
+		(color 0 0 0 0)
+	)
+	(junction
+		(at 129.54 182.88)
 		(diameter 0)
 		(color 0 0 0 0)
@@
 	)
 	(junction
-		(at 128.905 177.8)
-		(diameter 0)
-		(color 0 0 0 0)
-	)
-	(junction
 		(at 121.285 182.88)
 		(diameter 0)
@@
 	(wire
 		(pts
-			(xy 134.62 182.88) (xy 128.905 182.88)
+			(xy 134.62 182.88) (xy 129.54 182.88)
 		)
 		(stroke
@@
 	(wire
 		(pts
-			(xy 121.285 182.88) (xy 128.905 182.88)
+			(xy 121.285 182.88) (xy 129.54 182.88)
 		)
 		(stroke
@@
 	(wire
 		(pts
-			(xy 134.62 177.8) (xy 128.905 177.8)
+			(xy 134.62 177.8) (xy 129.54 177.8)
 		)
 		(stroke
@@
 	(wire
 		(pts
-			(xy 121.285 177.8) (xy 128.905 177.8)
+			(xy 121.285 177.8) (xy 129.54 177.8)
 		)
 		(stroke
@@
 	(symbol
 		(lib_id "Device:C_Small")
-		(at 128.905 180.34 0)
+		(at 129.54 180.34 0)
 		(unit 1)
 		(exclude_from_sim no)
@@
 		(dnp no)
 		(property "Reference" "C303"
-			(at 127.635 176.53 0)
+			(at 128.27 176.53 0)
 			(effects
 				(font
@@
 		)
 		(property "Value" "100n"
-			(at 127 184.15 0)
+			(at 127.635 184.15 0)
 			(effects
 				(font
@@
 		)
 		(property "Footprint" "A_Device:C_0603"
-			(at 128.905 180.34 0)
+			(at 129.54 180.34 0)
 			(effects
 				(font
@@
 		)
 		(property "Datasheet" "~"
-			(at 128.905 180.34 0)
+			(at 129.54 180.34 0)
 			(effects
 				(font
@@
 		)
 		(property "Description" ""
-			(at 128.905 180.34 0)
+			(at 129.54 180.34 0)
 			(effects
 				(font
@@
 		)
 		(property "LCSC" "C14663"
-			(at 128.905 180.34 0)
+			(at 129.54 180.34 0)
 			(effects
 				(font
@@
 		)
 		(property "JLCS" ""
-			(at 128.905 180.34 0)
-			(effects
-				(font
+			(at 129.54 180.34 0)
+			(effects
+				(font
