File: PCB/Robobuoy-Top-v2_1/Robobuoy-Top-v2_1.kicad_pcb (KiCad board)
At the start: 4 copper layers, 80 x 46 mm, 99 parts, among them J101 Prog, J102 Conn_01x06_Socket, J103 GPS, J201 CHRG/DATA, Q101 AO3400A, Q102 AO3400A, Q117 MMBT3904, Q201 MMBT3904, Q203 AO3400A, Q204 AO3401A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

Commit message: Some mods
Parts:
- C201, C202, C203, C204: footprint A_Device:C_1206_(1.6) -> Capacitor_SMD:C_1206_3216Metric
- U201: value LM1117DT-3.3 -> LM1117S-3.3; footprint Package_TO_SOT_SMD:TO-252-3_TabPin2 -> A_IC_SOT:SOT223
- moved U201 1.68 mm to (105.6, 70.9)
- moved C203 0.09 mm to (145.0, 67.4)
- moved R106 0.08 mm to (146.9, 67.5)
- moved C201 0.06 mm to (140.3, 67.4)
