File: PCB/Robobuoy-Top-v2_1/PSU_sch.kicad_sch (KiCad schematic)
At the start: 59 parts, among them J201 CHRG/DATA, Q117 MMBT3904, Q201 MMBT3904, Q203 AO3400A, Q204 AO3401A, SW201 On/Off, U201 LM1117DT-3.3, U202 LMR16020PDDA

Commit message: Some mods
Parts:
- C201, C202, C203, C204: footprint A_Device:C_1206_(1.6) -> Capacitor_SMD:C_1206_3216Metric
- U201: value LM1117DT-3.3 -> LM1117S-3.3; footprint Package_TO_SOT_SMD:TO-252-3_TabPin2 -> A_IC_SOT:SOT223; LCSC (none) -> C126027

Commit message: Loads of cahnges. Serial working stabile now (one resistor hardware mod) Ack hadled correct now. Less lora messsages
Other:
- note added: "1K"
Changed lines of the file:
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@@
+		)
+	)
+	(text "1K"
+		(exclude_from_sim no)
+		(at 84.836 92.456 0)
+		(effects
+			(font
+				(size 1.27 1.27)
+			)
 		)
 	)

Commit message: Many changes
Parts:
- added R207: 1K, A_Device:R_0603, symbol Device:R
Connections:
- net GND: now also R207.1
- net at Q201.1 (B), R109.2: now also R207.2
Other:
- note added: "New"
- note added: "must be 1K"
- note removed: "1K"
- moved on the sheet: R109, R111
