File: PCB/Robobuoy-Sub-Round-v2_0/Robobuoy-Sub-Round-v2_0.kicad_pcb (KiCad board)
At the start: 4 copper layers, 58.7 x 66.2 mm, 120 parts, among them J101 Prog, J201 ACCU, J202 CHRG/DATA, J301 ESC, J302 ESC_PWR, J401 ESC, J402 ESC_PWR, Q101 AO3400A, Q201 AO3400A, Q202 AO3401A, Q301 AO3400A, Q302 AO3401A, Q303 AO3401A, Q304 AO3401A, Q305 AO3401A, Q306 AO3401A, Q307 AO3401A, Q401 AO3400A, Q402 AO3401A, Q403 AO3401A, Q404 AO3401A, Q405 AO3401A, Q406 AO3401A, Q407 AO3401A, SW101 ~{RESET}, SW102 MODE, SW201 On/Off, U101 ESP32-WROOM-32E_(visible_peri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, U102 LSM303AGRTR, U103 USBLC6-4SC6, U201 TPS5430DDAR, U301 SN74LV1T34DBV, U401 SN74LV1T34DBV

Commit message: PCP's finsehd for production.
Parts:
- J201: value ACCU -> BATT
Routing:
- net EN: track 42.5 -> 40.0 mm, vias 0 -> 1
- net GND: track 189.0 -> 186.9 mm, vias 40 -> 94
- net +3.3V: track 228.5 -> 226.6 mm
- net Net-(U201-Vsens): track 13.1 -> 11.8 mm
- net /CPU/COM: track 51.0 -> 52.0 mm
- net BUZZER: track 17.2 -> 17.9 mm
- net Net-(J401-Pin_2): track 17.0 -> 16.4 mm
- net Vbatt: track 99.6 -> 99.0 mm
- net Net-(D204-K): track 11.3 -> 10.7 mm
- net Net-(J401-Pin_1): track 8.79 -> 8.28 mm
- added copper zone on B.Cu, net GND
Other:
- board text added: "+"
- board text added: "+25V"
- board text added: "-"
- board text added: "5V"
- board text added: "Compass"
- board text added: "D"
- board text added: "DR0 GND 3.3V"
- board text added: "ESC"
- board text added: "ESC PWR"
- board text added: "GND"
- board text added: "NICE ENGINEERING"
- board text added: "NicE Engineering"
- board text added: "OFF"
- board text added: "ON"
- board text added: "ON OFF"
- board text added: "PWM"
- board text added: "RESET"
- board text added: "ROBOBUOY SUB V2.0"
- board text added: "RX TX EN"
- board text added: "VBATT"
- board text added: "VIN"
- board text added: "X"
- board text added: "Y"
- board text added: "Z"
