File: PCB/Robobuoy_BMS_S6_V1_0/Robobuoy_BMS_S6_V1_0.kicad_sch (KiCad schematic)
At the start: 104 parts, among them J101 Balance, J102 Balance, J306 LiPo S6, Q102 AO3400A, Q103 AO3400A, Q104 AO3400A, Q105 AO3400A, Q106 AO3400A, Q107 AO3400A, Q108 AO3400A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

Commit message: PCB adjustmend Sub V3.0
Parts:
- added TP110: B1, A_Misc:TestPad_4x6, symbol Connector:TestPoint_Small
- added TP111: B2, A_Misc:TestPad_4x6, symbol Connector:TestPoint_Small
- added TP112: B3, A_Misc:TestPad_4x6, symbol Connector:TestPoint_Small
- added TP113: B4, A_Misc:TestPad_4x6, symbol Connector:TestPoint_Small
- added TP114: B5, A_Misc:TestPad_4x6, symbol Connector:TestPoint_Small
Connections:
- net B1: now also TP110.1
- net B2: now also TP111.1
- net B3: now also TP112.1
- net B4: now also TP113.1
- net B5: now also TP114.1

Commit message: Small changes on pcb
Parts:
- J101, J102: now not fitted
Connections:
- no-connect marks 5 -> 11
Changed lines of the file:
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@@
 	)
 	(junction
+		(at 368.3 153.67)
+		(diameter 0)
+		(color 0 0 0 0)
+	)
+	(junction
 		(at 101.6 193.04)
 		(diameter 0)
@@
 	)
 	(junction
+		(at 368.3 163.83)
+		(diameter 0)
+		(color 0 0 0 0)
+	)
+	(junction
 		(at 153.67 193.04)
 		(diameter 0)
@@
 	)
 	(no_connect
+		(at 121.92 205.74)
+	)
+	(no_connect
 		(at 227.33 187.96)
 	)
 	(no_connect
+		(at 121.92 104.14)
+	)
+	(no_connect
 		(at 227.33 86.36)
 	)
@@
 	)
 	(no_connect
+		(at 121.92 78.74)
+	)
+	(no_connect
 		(at 227.33 162.56)
 	)
 	(no_connect
+		(at 121.92 154.94)
+	)
+	(no_connect
 		(at 227.33 111.76)
 	)
+	(no_connect
+		(at 121.92 129.54)
+	)
+	(no_connect
+		(at 121.92 180.34)
+	)
 	(wire
 		(pts
@@
 	(wire
 		(pts
+			(xy 368.3 153.67) (xy 374.65 153.67)
+		)
+		(stroke
+			(width 0)
+			(type default)
+		)
+	)
+	(wire
+		(pts
 			(xy 256.54 114.3) (xy 256.54 121.92)
 		)
@@
 	(wire
 		(pts
-			(xy 360.68 163.83) (xy 374.65 163.83)
+			(xy 360.68 163.83) (xy 368.3 163.83)
 		)
 		(stroke
@@
 	(wire
 		(pts
-			(xy 360.68 153.67) (xy 374.65 153.67)
+			(xy 360.68 153.67) (xy 368.3 153.67)
 		)
 		(stroke
@@
 	(wire
 		(pts
+			(xy 368.3 163.83) (xy 374.65 163.83)
+		)
+		(stroke
+			(width 0)
+			(type default)
+		)
+	)
+	(wire
+		(pts
 			(xy 66.04 215.9) (xy 80.01 215.9)
 		)
@@
 		(in_bom yes)
 		(on_board yes)
-		(dnp no)
+		(dnp yes)
 		(property "Reference" "J102"
 			(at 382.27 114.3001 0)
@@
 	)
 	(symbol
+		(lib_id "power:PWR_FLAG")
+		(at 368.3 163.83 0)
+		(unit 1)
+		(exclude_from_sim no)
+		(in_bom yes)
+		(on_board yes)
+		(dnp no)
+		(fields_autoplaced yes)
+		(property "Reference" "#FLG0102"
+			(at 368.3 161.925 0)
+			(effects
+				(font
+					(size 1.27 1.27)
+				)
+				(hide yes)
+			)
+		)
+		(property "Value" "PWR_FLAG"
+			(at 368.3 158.75 0)
+			(effects
+				(font
+					(size 1.27 1.27)
+				)
+				(hide yes)
+			)
+		)
+		(property "Footprint" ""
+			(at 368.3 163.83 0)
+			(effects
+				(font
+					(size 1.27 1.27)
+				)
+				(hide yes)
+			)
+		)
+		(property "Datasheet" "~"
+			(at 368.3 163.83 0)
+			(effects
+				(font
+					(size 1.27 1.27)
+				)
+				(hide yes)
+			)
+		)
+		(property "Description" "Special symbol for telling ERC where power comes from"
+			(at 368.3 163.83 0)
+			(effects
+				(font
+					(size 1.27 1.27)
+				)
+				(hide yes)
+			)
+		)
+		(pin "1"
+		)
+		(instances
+			(project ""
+				(path "/1f52533e-1c9e-4a55-ac43-3d9bafbde785"
+					(reference "#FLG0102")
+					(unit 1)
+				)
+			)
+		)
+	)
+	(symbol
 		(lib_id "PCM_JLCPCB-Transistors:NMOS,AO3400A")
 		(at 81.28 99.06 180)
@@
 		(in_bom yes)
 		(on_board yes)
-		(dnp no)
+		(dnp yes)
 		(property "Reference" "J101"
 			(at 364.49 114.3001 0)
@@
 					(unit 1)
 				)
+			)
+		)
+	)
+	(symbol
+		(lib_id "power:PWR_FLAG")
+		(at 368.3 153.67 0)
+		(unit 1)
+		(exclude_from_sim no)
+		(in_bom yes)
+		(on_board yes)
+		(dnp no)
+		(fields_autoplaced yes)
+		(property "Reference" "#FLG0101"
+			(at 368.3 151.765 0)
+			(effects
+				(font
+					(size 1.27 1.27)
+				)
+				(hide yes)
+			)
+		)
+		(property "Value" "PWR_FLAG"
+			(at 368.3 148.59 0)
+			(effects
+				(font
+					(size 1.27 1.27)
+				)
+				(hide yes)
+			)
+		)
+		(property "Footprint" ""
+			(at 368.3 153.67 0)
+			(effects
+				(font
+					(size 1.27 1.27)
+				)
+				(hide yes)
+			)
+		)
+		(property "Datasheet" "~"
+			(at 368.3 153.67 0)
+			(effects
+				(font
+					(size 1.27 1.27)
+				)
+				(hide yes)
+			)
+		)
+		(property "Description" "Special symbol for telling ERC where power comes from"
+			(at 368.3 153.67 0)
+			(effects
+				(font
+					(size 1.27 1.27)
+				)
+				(hide yes)
+			)
+		)
+		(pin "1"
+		)
+		(instances
+			(project ""
+				(path "/1f52533e-1c9e-4a55-ac43-3d9bafbde785"
+					(reference "#FLG0101")
+					(unit 1)
+				)

Commit message: Heel veel AI veranderingen.
Parts:
- R149, R150, R151, R152, R153: value 24K -> 27K
Changed lines of the file:
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@@
 			)
 		)
-		(property "Value" "24K"
+		(property "Value" "27K"
 			(at 234.442 118.618 0)
 			(effects
@@
 			)
 		)
-		(property "Value" "24K"
+		(property "Value" "27K"
 			(at 231.902 93.218 0)
 			(effects
@@
 			)
 		)
-		(property "Value" "24K"
+		(property "Value" "27K"
 			(at 234.442 194.818 0)
 			(effects
@@
 			)
 		)
-		(property "Value" "24K"
+		(property "Value" "27K"
 			(at 234.442 169.418 0)
 			(effects
@@
 			)
 		)
-		(property "Value" "24K"
+		(property "Value" "27K"
 			(at 234.442 144.018 0)
 			(effects

Commit message: docs: update PCB schematics and add ICM20948 datasheet
Other:
- note added: "Moet Pmos worden"
Changed lines of the file:
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@@
+		)
+	)
+	(text "Moet Pmos worden"
+		(exclude_from_sim no)
+		(at 74.295 60.325 0)
+		(effects
+			(font
+				(size 1.27 1.27)
+			)
 		)
 	)
