File: PCBA_Robobouoy-V4.0/Robobuoy-Top-CPU-V4.0.kicad_sch (KiCad schematic)
At the start: 40 parts, among them J501 Prog, J502 LIGHT/BUTTON, J503 GPS, J504 LEDSTRIP, J506 Conn_01x08_Pin, Q501 AO3400A, Q502 AO3400A, U501 ESP32-WROOM-32E_(visible_peri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, U502 Ai-Thinker-Ra-02

Commit message: Some pcb changes
Connections:
- net RADIO_6: no longer J506.8 (Pin_8)
- net CS_2: now reaches U501.13 (MTMS/SCK/CLK/GPIO14)
- net CS_2: now also J506.8 (Pin_8)
Changed lines of the file:
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@@
+	(wire
+		(pts
+			(xy 205.74 85.09) (xy 224.79 85.09)
+		)
+		(stroke
+			(width 0)
+			(type default)
+		)
+	)
 	(wire
 		(pts
@@
 		)
 	)
+	(label "CS_2"
+		(at 219.71 85.09 0)
+		(effects
+			(font
+				(size 1.27 1.27)
+			)
+			(justify left bottom)
+		)
+	)
 	(label "RADIO_3"
 		(at 66.04 43.18 0)
@@
 		)
 	)
-	(label "RADIO_6"
-		(at 66.04 50.8 0)
-		(effects
-			(font
-				(size 1.27 1.27)
-			)
-			(justify left bottom)
-		)
-	)
 	(label "RADIO_1"
 		(at 217.17 97.79 0)
 		(effects
 			(font
+				(size 1.27 1.27)
+			)
+			(justify left bottom)
+		)
+	)
+	(label "CS_2"
+		(at 68.58 50.8 0)
+		(effects
+			(font
